Commit message: Update model

File: ros2_ws/src/simple_3r_arm/simple_3r_arm_description/urdf/simple_3r_arm_description.urdf.xacro (robot description, xacro)
@@ -33,5 +33,5 @@
           <box size="${width} ${width} ${heightBase}"/>
         </geometry>
-        <material name="orange"/>
+        <material name="black"/>
       </visual>
       <inertial>
@@ -47,5 +47,5 @@
       <parent link="${prefix}base_link"/>
       <child link="${prefix}link1"/>
-      <origin xyz="0 0 ${heightBase - axel_offset}" rpy="0 0 0"/>
+      <origin xyz="0 0 ${heightBase}" rpy="0 0 0"/>
       <axis xyz="0 0 1"/>
       <dynamics damping="0.7"/>
@@ -53,5 +53,5 @@
     <link name="${prefix}link1">
       <collision>
-        <origin xyz="0 0 ${height1/2 - axel_offset}" rpy="0 0 0"/>
+        <origin xyz="0 0 ${height1/2}" rpy="0 0 0"/>
         <geometry>
           <box size="${width} ${width} ${height1}"/>
@@ -59,12 +59,12 @@
       </collision>
       <visual>
-        <origin xyz="0 0 ${height1/2 - axel_offset}" rpy="0 0 0"/>
+        <origin xyz="0 0 ${height1/2}" rpy="0 0 0"/>
         <geometry>
           <box size="${width} ${width} ${height1}"/>
         </geometry>
-        <material name="yellow"/>
+        <material name="orange"/>
       </visual>
       <inertial>
-        <origin xyz="0 0 ${height1/2 - axel_offset}" rpy="0 0 0"/>
+        <origin xyz="0 0 ${height1/2}" rpy="0 0 0"/>
         <mass value="${mass}"/>
         <inertia ixx="${mass / 12.0 * (width*width + height1*height1)}" ixy="0.0" ixz="0.0"
@@ -77,5 +77,5 @@
       <parent link="${prefix}link1"/>
       <child link="${prefix}link2"/>
-      <origin xyz="0 ${width} ${height1 - axel_offset*2}" rpy="0 0 0"/>
+      <origin xyz="0 ${width} ${height1 - axel_offset}" rpy="0 0 0"/>
       <axis xyz="0 1 0"/>
       <dynamics damping="0.7"/>
@@ -83,5 +83,5 @@
     <link name="${prefix}link2">
       <collision>
-        <origin xyz="0 0 ${height2/2 - axel_offset}" rpy="0 0 0"/>
+        <origin xyz="0 0 ${height2/2}" rpy="0 0 0"/>
         <geometry>
           <box size="${width} ${width} ${height2}"/>
@@ -89,12 +89,12 @@
       </collision>
       <visual>
-        <origin xyz="0 0 ${height2/2 - axel_offset}" rpy="0 0 0"/>
+        <origin xyz="0 0 ${height2/2}" rpy="0 0 0"/>
         <geometry>
           <box size="${width} ${width} ${height2}"/>
         </geometry>
-        <material name="orange"/>
+        <material name="yellow"/>
       </visual>
       <inertial>
-        <origin xyz="0 0 ${height2/2 - axel_offset}" rpy="0 0 0"/>
+        <origin xyz="0 0 ${height2/2}" rpy="0 0 0"/>
         <mass value="${mass}"/>
         <inertia ixx="${mass / 12.0 * (width*width + height2*height2)}" ixy="0.0" ixz="0.0"
@@ -107,5 +107,5 @@
       <parent link="${prefix}link2"/>
       <child link="${prefix}link3"/>
-      <origin xyz="0 ${width} ${height1 - axel_offset*2}" rpy="0 0 0"/>
+      <origin xyz="0 -${width} ${height1 - axel_offset}" rpy="0 0 0"/>
       <axis xyz="0 1 0"/>
       <dynamics damping="0.7"/>
@@ -113,18 +113,18 @@
     <link name="${prefix}link3">
       <collision>
-        <origin xyz="0 0 ${height3/2 - axel_offset}" rpy="0 0 0"/>
+        <origin xyz="0 0 ${height3/2}" rpy="0 0 0"/>
         <geometry>
-          <box size="${width} ${width} ${height3}"/>
+          <box size="${width} -${width} ${height3}"/>
         </geometry>
       </collision>
       <visual>
-        <origin xyz="0 0 ${height3/2 - axel_offset}" rpy="0 0 0"/>
+        <origin xyz="0 0 ${height3/2}" rpy="0 0 0"/>
         <geometry>
-          <box size="${width} ${width} ${height3}"/>
+          <box size="${width} -${width} ${height3}"/>
         </geometry>
-        <material name="orange"/>
+        <material name="green"/>
       </visual>
       <inertial>
-        <origin xyz="0 0 ${height3/2 - axel_offset}" rpy="0 0 0"/>
+        <origin xyz="0 0 ${height3/2}" rpy="0 0 0"/>
         <mass value="${mass}"/>
         <inertia ixx="${mass / 12.0 * (width*width + height3*height3)}" ixy="0.0" ixz="0.0"

Commit message: Update simpl3_3r_arm  model

File: ros2_ws/src/simple_3r_arm/simple_3r_arm_description/urdf/simple_3r_arm_description.urdf.xacro (robot description, xacro)
@@ -9,8 +9,8 @@
     <!-- Constants for robot dimensions -->
     <xacro:property name="mass" value="1" /> <!-- arbitrary value for mass -->
-    <xacro:property name="heightBase" value="2" /> <!-- Base Link -->
-    <xacro:property name="height1" value="1" /> <!-- Link 1 -->
-    <xacro:property name="height2" value="1" /> <!-- Link 2 -->
-    <xacro:property name="height3" value="1" /> <!-- Link 3 -->
+    <xacro:property name="lengthBase" value="2" /> <!-- Base Link -->
+    <xacro:property name="length1" value="1" /> <!-- Link 1 -->
+    <xacro:property name="length2" value="1" /> <!-- Link 2 -->
+    <xacro:property name="length3" value="1" /> <!-- Link 3 -->
     <xacro:property name="width" value="0.1" /> <!-- Square dimensions (widthxwidth) of beams -->
     <xacro:property name="axel_offset" value="0.05" /> <!-- Space btw top of beam and the each joint -->
@@ -23,21 +23,21 @@
     <link name="${prefix}base_link">
       <collision>
-        <origin xyz="0 0 ${heightBase/2}" rpy="0 0 0"/>
+        <origin xyz="0 0 ${lengthBase/2}" rpy="0 0 0"/>
         <geometry>
-          <box size="${width} ${width} ${heightBase}"/>
+          <box size="${width} ${width} ${lengthBase}"/>
         </geometry>
       </collision>
       <visual>
-        <origin xyz="0 0 ${heightBase/2}" rpy="0 0 0"/>
+        <origin xyz="0 0 ${lengthBase/2}" rpy="0 0 0"/>
         <geometry>
-          <box size="${width} ${width} ${heightBase}"/>
+          <box size="${width} ${width} ${lengthBase}"/>
         </geometry>
         <material name="black"/>
       </visual>
       <inertial>
-        <origin xyz="0 0 ${heightBase/2}" rpy="0 0 0"/>
+        <origin xyz="0 0 ${lengthBase/2}" rpy="0 0 0"/>
         <mass value="${mass}"/>
-        <inertia ixx="${mass / 12.0 * (width*width + heightBase*heightBase)}" ixy="0.0" ixz="0.0"
-                 iyy="${mass / 12.0 * (heightBase*heightBase + width*width)}" iyz="0.0"
+        <inertia ixx="${mass / 12.0 * (width*width + lengthBase*lengthBase)}" ixy="0.0" ixz="0.0"
+                 iyy="${mass / 12.0 * (lengthBase*lengthBase + width*width)}" iyz="0.0"
                  izz="${mass / 12.0 * (width*width + width*width)}"/>
       </inertial>
@@ -47,5 +47,5 @@
       <parent link="${prefix}base_link"/>
       <child link="${prefix}link1"/>
-      <origin xyz="0 0 ${heightBase}" rpy="0 0 0"/>
+      <origin xyz="0 0 ${lengthBase}" rpy="0 0 0"/>
       <axis xyz="0 0 1"/>
       <dynamics damping="0.7"/>
@@ -53,21 +53,21 @@
     <link name="${prefix}link1">
       <collision>
-        <origin xyz="0 0 ${height1/2}" rpy="0 0 0"/>
+        <origin xyz="0 0 ${length1/2}" rpy="0 0 0"/>
         <geometry>
-          <box size="${width} ${width} ${height1}"/>
+          <box size="${width} ${width} ${length1}"/>
         </geometry>
       </collision>
       <visual>
-        <origin xyz="0 0 ${height1/2}" rpy="0 0 0"/>
+        <origin xyz="0 0 ${length1/2}" rpy="0 0 0"/>
         <geometry>
-          <box size="${width} ${width} ${height1}"/>
+          <box size="${width} ${width} ${length1}"/>
         </geometry>
         <material name="orange"/>
       </visual>
       <inertial>
-        <origin xyz="0 0 ${height1/2}" rpy="0 0 0"/>
+        <origin xyz="0 0 ${length1/2}" rpy="0 0 0"/>
         <mass value="${mass}"/>
-        <inertia ixx="${mass / 12.0 * (width*width + height1*height1)}" ixy="0.0" ixz="0.0"
-                 iyy="${mass / 12.0 * (height1*height1 + width*width)}" iyz="0.0"
+        <inertia ixx="${mass / 12.0 * (width*width + length1*length1)}" ixy="0.0" ixz="0.0"
+                 iyy="${mass / 12.0 * (length1*length1 + width*width)}" iyz="0.0"
                  izz="${mass / 12.0 * (width*width + width*width)}"/>
       </inertial>
@@ -77,5 +77,5 @@
       <parent link="${prefix}link1"/>
       <child link="${prefix}link2"/>
-      <origin xyz="0 ${width} ${height1 - axel_offset}" rpy="0 0 0"/>
+      <origin xyz="0 ${width} ${length1}" rpy="0 0 0"/>
       <axis xyz="0 1 0"/>
       <dynamics damping="0.7"/>
@@ -83,21 +83,21 @@
     <link name="${prefix}link2">
       <collision>
-        <origin xyz="0 0 ${height2/2}" rpy="0 0 0"/>
+        <origin xyz="${length2/2} 0 0" rpy="0 ${pi/2} 0"/>
         <geometry>
-          <box size="${width} ${width} ${height2}"/>
+          <box size="${width} ${width} ${length2}"/>
         </geometry>
       </collision>
       <visual>
-        <origin xyz="0 0 ${height2/2}" rpy="0 0 0"/>
+        <origin xyz="${length2/2} 0 0" rpy="0 ${pi/2} 0"/>
         <geometry>
-          <box size="${width} ${width} ${height2}"/>
+          <box size="${width} ${width} ${length2}"/>
         </geometry>
         <material name="yellow"/>
       </visual>
       <inertial>
-        <origin xyz="0 0 ${height2/2}" rpy="0 0 0"/>
+        <origin xyz="${length2/2} 0 0" rpy="0 ${pi/2} 0"/>
         <mass value="${mass}"/>
-        <inertia ixx="${mass / 12.0 * (width*width + height2*height2)}" ixy="0.0" ixz="0.0"
-                 iyy="${mass / 12.0 * (height2*height2 + width*width)}" iyz="0.0"
+        <inertia ixx="${mass / 12.0 * (width*width + length2*length2)}" ixy="0.0" ixz="0.0"
+                 iyy="${mass / 12.0 * (length2*length2 + width*width)}" iyz="0.0"
                  izz="${mass / 12.0 * (width*width + width*width)}"/>
       </inertial>
@@ -107,5 +107,5 @@
       <parent link="${prefix}link2"/>
       <child link="${prefix}link3"/>
-      <origin xyz="0 -${width} ${height1 - axel_offset}" rpy="0 0 0"/>
+      <origin xyz="${length2} -${width} 0" rpy="0 0 0"/>
       <axis xyz="0 1 0"/>
       <dynamics damping="0.7"/>
@@ -113,21 +113,21 @@
     <link name="${prefix}link3">
       <collision>
-        <origin xyz="0 0 ${height3/2}" rpy="0 0 0"/>
+        <origin xyz="${length3/2} 0 0" rpy="0 ${pi/2} 0"/>
         <geometry>
-          <box size="${width} -${width} ${height3}"/>
+          <box size="${width} -${width} ${length3}"/>
         </geometry>
       </collision>
       <visual>
-        <origin xyz="0 0 ${height3/2}" rpy="0 0 0"/>
+        <origin xyz="${length3/2} 0 0" rpy="0 ${pi/2} 0"/>
         <geometry>
-          <box size="${width} -${width} ${height3}"/>
+          <box size="${width} -${width} ${length3}"/>
         </geometry>
         <material name="green"/>
       </visual>
       <inertial>
-        <origin xyz="0 0 ${height3/2}" rpy="0 0 0"/>
+        <origin xyz="${length3/2} 0 0" rpy="0 ${pi/2} 0"/>
         <mass value="${mass}"/>
-        <inertia ixx="${mass / 12.0 * (width*width + height3*height3)}" ixy="0.0" ixz="0.0"
-                 iyy="${mass / 12.0 * (height3*height3 + width*width)}" iyz="0.0"
+        <inertia ixx="${mass / 12.0 * (width*width + length3*length3)}" ixy="0.0" ixz="0.0"
+                 iyy="${mass / 12.0 * (length3*length3 + width*width)}" iyz="0.0"
                  izz="${mass / 12.0 * (width*width + width*width)}"/>
       </inertial>
